File: PCB/Akita/LinuxSiP.sch (KiCad schematic (older format))
At the start: 0 parts

Commit message: Add Octavo SiP to project
Lifted from PocketBeagle design.

Signed-off-by: Michael Welling <mwelling@ieee.org>
Parts:
- added U? (x6): OSD3358-512M-BSM, OSD335X-BGA-256, symbol Akita_Pro_Library:OSD3358-512M-BSM
Changed lines of the file:
@@
 EELAYER 29 0
 EELAYER END
-$Descr A4 11693 8268
+$Descr A2 23386 16535
 encoding utf-8
 Sheet 4 7
@@
 Comment4 ""
 $EndDescr
+$Comp
+L Akita_Pro_Library:OSD3358-512M-BSM U?
+U 1 1 5D3D42E3
+P 3700 8600
+F 0 "U?" H 4900 15554 45  0000 C CNN
+F 1 "OSD3358-512M-BSM" H 4900 15470 45  0000 C CNN
+F 2 "OSD335X-BGA-256" H 3730 8750 20  0001 C CNN
+F 3 "" H 3700 8600 60  0001 C CNN
+	1    3700 8600
+	1    0    0    -1
+$EndComp
+$Comp
+L Akita_Pro_Library:OSD3358-512M-BSM U?
+U 2 1 5D3DB153
+P 10225 6475
+F 0 "U?" H 11325 11329 45  0000 C CNN
+F 1 "OSD3358-512M-BSM" H 11325 11245 45  0000 C CNN
+F 2 "OSD335X-BGA-256" H 10255 6625 20  0001 C CNN
+F 3 "" H 10225 6475 60  0001 C CNN
+	2    10225 6475
+	1    0    0    -1
+$EndComp
+$Comp
+L Akita_Pro_Library:OSD3358-512M-BSM U?
+U 3 1 5D3E5D84
+P 17100 6800
+F 0 "U?" H 18250 11854 45  0000 C CNN
+F 1 "OSD3358-512M-BSM" H 18250 11770 45  0000 C CNN
+F 2 "OSD335X-BGA-256" H 17130 6950 20  0001 C CNN
+F 3 "" H 17100 6800 60  0001 C CNN
+	3    17100 6800
+	1    0    0    -1
+$EndComp
+$Comp
+L Akita_Pro_Library:OSD3358-512M-BSM U?
+U 4 1 5D3EE26B
+P 3675 13700
+F 0 "U?" H 4675 16554 45  0000 C CNN
+F 1 "OSD3358-512M-BSM" H 4675 16470 45  0000 C CNN
+F 2 "OSD335X-BGA-256" H 3705 13850 20  0001 C CNN
+F 3 "" H 3675 13700 60  0001 C CNN
+	4    3675 13700
+	1    0    0    -1
+$EndComp
+$Comp
+L Akita_Pro_Library:OSD3358-512M-BSM U?
+U 5 1 5D3F7AED
+P 11400 12325
+F 0 "U?" H 11400 13779 45  0000 C CNN
+F 1 "OSD3358-512M-BSM" H 11400 13695 45  0000 C CNN
+F 2 "OSD335X-BGA-256" H 11430 12475 20  0001 C CNN
+F 3 "" H 11400 12325 60  0001 C CNN
+	5    11400 12325
+	1    0    0    -1
+$EndComp
+$Comp
+L Akita_Pro_Library:OSD3358-512M-BSM U?
+U 6 1 5D402F53
+P 17250 13400
+F 0 "U?" H 18150 15454 45  0000 C CNN
+F 1 "OSD3358-512M-BSM" H 18150 15370 45  0000 C CNN
+F 2 "OSD335X-BGA-256" H 17280 13550 20  0001 C CNN
+F 3 "" H 17250 13400 60  0001 C CNN
+	6    17250 13400
+	1    0    0    -1
+$EndComp
 $EndSCHEMATC
